Commit message: feat: URDF 加入中央伸缩腿并接入弹簧插件与 leg_state 桥接

File: ros2_ws/src/quadcopter_description/urdf/quadcopter.urdf.xacro (robot description, xacro)
@@ -33,6 +33,16 @@
   <xacro:property name="arm_radius" value="0.002"/>
   <xacro:property name="motor_z" value="${body_z / 2.0 + motor_height / 2.0}"/>
-  <!-- Mass (kg); total = 0.027 -->
-  <xacro:property name="mass_base" value="0.016"/>
+  <!-- Hopcopter passive telescopic leg (paper Eq. 7 / table S2) -->
+  <xacro:property name="leg_length0" value="0.22"/>
+  <xacro:property name="leg_preload" value="0.0197"/>
+  <xacro:property name="mass_total" value="0.0348"/>
+  <xacro:property name="foot_mass" value="0.001"/>
+  <xacro:property name="k_over_m" value="5000.0"/>
+  <xacro:property name="f_c_over_m" value="12.7"/>
+  <xacro:property name="spring_k" value="${k_over_m * mass_total}"/>
+  <xacro:property name="spring_f_c" value="${f_c_over_m * mass_total}"/>
+  <!-- Mass (kg); total = 0.0348 = base + 4 props + foot -->
+  <xacro:property name="mass_base"
+                  value="${mass_total - 4.0 * mass_prop_link - foot_mass}"/>
   <xacro:property name="mass_prop_link" value="0.00275"/>
   <!-- Motor model (approximate, to be calibrated in task 6) -->
@@ -191,4 +201,46 @@
                        y="${body_y}" z="${body_z}"/>
   </link>
+  <!-- Central monopedal telescopic leg: foot_link slides along body z.
+       q = 0 corresponds to the rest length l0 = 0.22 m (mechanical stop);
+       compression moves the foot towards the body (q < 0). -->
+  <link name="foot_link">
+    <visual name="leg_rod">
+      <origin xyz="0 0 ${leg_length0 / 2.0}" rpy="0 0 0"/>
+      <geometry>
+        <cylinder radius="${leg_radius}" length="${leg_length0}"/>
+      </geometry>
+      <material name="black"/>
+    </visual>
+    <visual name="foot_tip">
+      <origin xyz="0 0 0" rpy="0 0 0"/>
+      <geometry>
+        <sphere radius="0.004"/>
+      </geometry>
+      <material name="gray"/>
+    </visual>
+    <collision name="foot_tip">
+      <origin xyz="0 0 0" rpy="0 0 0"/>
+      <geometry>
+        <sphere radius="0.004"/>
+      </geometry>
+    </collision>
+    <inertial>
+      <mass value="${foot_mass}"/>
+      <inertia
+        ixx="${0.4 * foot_mass * 0.004 * 0.004}"
+        ixy="0.0" ixz="0.0"
+        iyy="${0.4 * foot_mass * 0.004 * 0.004}"
+        iyz="0.0"
+        izz="${0.4 * foot_mass * 0.004 * 0.004}"/>
+    </inertial>
+  </link>
+  <joint name="leg_joint" type="prismatic">
+    <parent link="base_link"/>
+    <child link="foot_link"/>
+    <origin xyz="0 0 ${-leg_length0}" rpy="0 0 0"/>
+    <axis xyz="0 0 -1"/>
+    <limit lower="-0.16" upper="0.0" effort="100.0" velocity="10.0"/>
+    <dynamics damping="0.0" friction="0.0"/>
+  </joint>
   <xacro:motor_prop idx="0" x="${motor_xy}" y="${motor_xy}"
                     yaw="${yaw_0}" turning="ccw"/>
@@ -204,9 +256,26 @@
       filename="gz-sim-joint-state-publisher-system"
       name="gz::sim::systems::JointStatePublisher">
-      <update_rate>50</update_rate>
+      <update_rate>500</update_rate>
       <joint_name>prop0_joint</joint_name>
       <joint_name>prop1_joint</joint_name>
       <joint_name>prop2_joint</joint_name>
       <joint_name>prop3_joint</joint_name>
+      <joint_name>leg_joint</joint_name>
+    </plugin>
+  </gazebo>
+  <!-- Passive spring-damper leg (paper Eq. 7, custom gz-sim system plugin).
+       Forces are applied at the physics rate; state is published at 1 kHz. -->
+  <gazebo>
+    <plugin
+      filename="libspring_damper_leg_system.so"
+      name="quadcopter_gz_plugins::SpringDamperLegSystem">
+      <leg_joint>leg_joint</leg_joint>
+      <foot_link>foot_link</foot_link>
+      <k>${spring_k}</k>
+      <f_c>${spring_f_c}</f_c>
+      <l_p>${leg_preload}</l_p>
+      <l0>${leg_length0}</l0>
+      <vel_eps>0.02</vel_eps>
+      <topic>/model/quadcopter/leg_state</topic>
     </plugin>
   </gazebo>

Commit message: feat: 姿态控制节点/IMU与电机桥接/launch 及任务六验证脚本

File: ros2_ws/src/quadcopter_description/urdf/quadcopter.urdf.xacro (robot description, xacro)
@@ -46,8 +46,11 @@
                   value="${mass_total - 4.0 * mass_prop_link - foot_mass}"/>
   <xacro:property name="mass_prop_link" value="0.00275"/>
-  <!-- Motor model (approximate, to be calibrated in task 6) -->
+  <!-- Motor model (calibrated in task 6):
+       force = motor_constant * speed^2,  torque = moment_constant * force.
+       Hover needs ~2/3 max speed; moment_constant matches the Crazyflie
+       torque/thrust ratio (~0.006 m). -->
   <xacro:property name="max_rot_velocity" value="2200.0"/>
   <xacro:property name="motor_constant" value="3.0e-8"/>
-  <xacro:property name="moment_constant" value="3.0e-5"/>
+  <xacro:property name="moment_constant" value="0.006"/>
   <xacro:property name="time_constant_up" value="0.02"/>
   <xacro:property name="time_constant_down" value="0.04"/>
@@ -243,10 +246,12 @@
     <dynamics damping="0.0" friction="0.0"/>
   </joint>
+  <!-- Adjacent rotors spin in opposite directions so roll and yaw torques are
+       independent (standard X4 layout: CCW, CW, CCW, CW). -->
   <xacro:motor_prop idx="0" x="${motor_xy}" y="${motor_xy}"
                     yaw="${yaw_0}" turning="ccw"/>
   <xacro:motor_prop idx="1" x="${-motor_xy}" y="${motor_xy}"
-                    yaw="${yaw_1}" turning="ccw"/>
+                    yaw="${yaw_1}" turning="cw"/>
   <xacro:motor_prop idx="2" x="${-motor_xy}" y="${-motor_xy}"
-                    yaw="${yaw_2}" turning="cw"/>
+                    yaw="${yaw_2}" turning="ccw"/>
   <xacro:motor_prop idx="3" x="${motor_xy}" y="${-motor_xy}"
                     yaw="${yaw_3}" turning="cw"/>
@@ -291,3 +296,17 @@
     </plugin>
   </gazebo>
+  <!-- IMU on the body: quaternion + angular velocity for the attitude loop -->
+  <gazebo reference="base_link">
+    <sensor name="imu_sensor" type="imu">
+      <always_on>1</always_on>
+      <update_rate>500</update_rate>
+      <visualize>false</visualize>
+      <imu>
+        <orientation_reference_frame>ENU</orientation_reference_frame>
+      </imu>
+      <plugin
+        filename="gz-sim-imu-system"
+        name="gz::sim::systems::Imu"/>
+    </sensor>
+  </gazebo>
 </robot>

Commit message: feat: Gazebo 气动稳定器系统插件（平板理论力矩、激活订阅）与 URDF/launch 接线

File: ros2_ws/src/quadcopter_description/urdf/quadcopter.urdf.xacro (robot description, xacro)
@@ -169,4 +169,16 @@
     </gazebo>
   </xacro:macro>
+  <!-- Aerodynamic stabilizer visual: three 39 cm^2 hinged plates (paper
+       Fig. 6A).  The plates are visual-only; the aerodynamic aligning
+       torque is applied by the dedicated gz-sim system plugin below. -->
+  <xacro:macro name="stabilizer_plate" params="idx angle">
+    <visual name="stab_plate_${idx}">
+      <origin xyz="0 0 ${body_z / 2.0 + 0.012}" rpy="0 ${pi / 2.0 - 0.30} ${angle}"/>
+      <geometry>
+        <box size="0.052 0.075 0.001"/>
+      </geometry>
+      <material name="prop_white"/>
+    </visual>
+  </xacro:macro>
   <!-- ================================ links ================================ -->
   <material name="black">
@@ -195,4 +207,7 @@
     <xacro:leg x="-0.028" y="-0.028"/>
     <xacro:leg x="0.028" y="-0.028"/>
+    <xacro:stabilizer_plate idx="0" angle="0"/>
+    <xacro:stabilizer_plate idx="1" angle="${2.0943951023931953}"/>
+    <xacro:stabilizer_plate idx="2" angle="${4.1887902047863905}"/>
     <collision name="body">
       <origin xyz="0 0 0" rpy="0 0 0"/>
@@ -285,4 +300,23 @@
     </plugin>
   </gazebo>
+  <!-- Active aerodynamic stabilizer (paper SM Eq. S33, custom gz-sim
+       system plugin).  The ROS controller publishes
+       /quadcopter/stabilizer_cmd (Bool); the launch file bridges it to the
+       plugin topic.  When active, the plugin applies the flat-plate
+       aligning torque computed from the body's own world velocity. -->
+  <gazebo>
+    <plugin
+      filename="libaerodynamic_stabilizer_system.so"
+      name="quadcopter_gz_plugins::AerodynamicStabilizerSystem">
+      <link_name>base_link</link_name>
+      <rho>1.2</rho>
+      <surface>0.0078</surface>
+      <k_eff>8.0</k_eff>
+      <moment_arm>0.06</moment_arm>
+      <speed_eps>0.05</speed_eps>
+      <topic>/model/quadcopter/stabilizer_active</topic>
+      <diag_topic>/model/quadcopter/stabilizer_state</diag_topic>
+    </plugin>
+  </gazebo>
   <!-- Publish the model pose (used by the RViz TF pipeline) -->
   <gazebo>
